Commit message: Recolor chassis and floor collision links
- Changed chassis_link material to chassis_orange (0.90 0.45 0.10)
- Changed floor_link material to floor_brown (0.40 0.26 0.13)
- Renamed both materials from the stale _grey names
- Kept the original alpha values so both stay semi-transparent

File: dofbot_description/urdf/chassis.xacro (robot description, xacro)
@@ -28,9 +28,9 @@
       floor_x_back:=-0.5
       floor_half_width:=0.35">
-    <material name="chassis_grey">
-      <color rgba="0.35 0.37 0.42 0.55"/>
+    <material name="chassis_orange">
+      <color rgba="0.90 0.45 0.10 0.55"/>
     </material>
-    <material name="floor_grey">
-      <color rgba="0.30 0.30 0.30 0.35"/>
+    <material name="floor_brown">
+      <color rgba="0.40 0.26 0.13 0.35"/>
     </material>
     <!-- Robot body: a z-axis cylinder behind the arm. URDF cylinders are
@@ -42,5 +42,5 @@
           <cylinder radius="${radius}" length="${height}"/>
         </geometry>
-        <material name="chassis_grey"/>
+        <material name="chassis_orange"/>
       </visual>
       <collision>
@@ -65,5 +65,5 @@
                      ${floor_thickness}"/>
         </geometry>
-        <material name="floor_grey"/>
+        <material name="floor_brown"/>
       </visual>
       <collision>
