Commit message: Select the floor height by measured surface type
- Replaced floor_z_top's RViz-fitted -0.015 with measured values
- Added DOFBOT_FLOOR (env var) choosing carpet 0.022 or hard floor 0.026
- Defaulted unset and unrecognised values to carpet, the safe direction
- Removed the resolved floor_z_top entry from Known open items

Co-Authored-By: Claude Opus 5 <noreply@anthropic.com>

File: dofbot_description/urdf/chassis.xacro (robot description, xacro)
@@ -11,10 +11,29 @@
   origin at the arm mounting plate (its underside is z=0).
   The floor is attached to base_link, not to the world, on purpose: the robot is
-  mobile, and the work surface is always the same fixed distance below the arm's
-  mounting plate. Hanging it off base_link keeps that true as the robot drives.
+  mobile, and the work surface stays a fixed distance below the arm's mounting
+  plate for as long as it stays on one surface. Hanging it off base_link keeps
+  that true as the robot drives. Change surface and the distance changes; see
+  DOFBOT_FLOOR below.
   Defaults are the values measured on the real robot and validated at runtime
   through the chassis_collision node (which this replaces).
 -->
 <robot xmlns:xacro="http://www.ros.org/wiki/xacro">
+  <!-- Which surface the robot is standing on. The wheels sink into a soft
+       floor, so the whole robot rides lower and the ground sits CLOSER to the
+       mounting plate. Measured 2026-08-25 from the plate's underside, which is
+       base_link z=0:
+         carpet      22 mm   Jim's office; where picking is tested
+         hard floor  26 mm   the contest surface
+       Unset or unrecognised gives carpet, and that is the SAFE way round.
+       22 mm models the ground HIGHER than a hard floor really is, so MoveIt
+       gives up the bottom 4 mm of reach. The reverse puts the collision plane
+       BELOW real carpet and lets the gripper plan into it.
+       An env var rather than a xacro:arg for the same reason as DOFBOT_GRIPPER
+       in dofbot.urdf: urdf_launch runs xacro with no arguments, and display,
+       mirror and gui_teleop all load the model through urdf_launch, so a
+       xacro:arg could never be overridden there. -->
+  <xacro:property name="floor_profile" value="$(optenv DOFBOT_FLOOR carpet)" />
+  <xacro:property name="ground_drop"
+                  value="${0.026 if floor_profile == 'hard' else 0.022}" />
   <xacro:macro name="dofbot_chassis" params="
       parent:=base_link
@@ -23,5 +42,5 @@
       back_offset:=0.265
       z_bottom:=0.003
-      floor_z_top:=-0.015
+      floor_z_top:=${-ground_drop}
       floor_thickness:=0.005
       floor_x_front:=0.35

Commit message: Re-pose init to clear the OAK-D's view, and correct the chassis radius
- Changed init (named state) to a lower, further-forward pose that clears the
  chassis OAK-D's view of a can on the floor, measured on the arm
- Applied the same pose to the SRDF group_state and initial_positions.yaml
- Raised arm3_Joint's URDF upper limit, which the new pose needs
- Changed JOINT_LIMITS (tuple) in dofbot_kinematics to match
- Changed the chassis cylinder radius to the pancake decks rather than the
  body's widest point, measured as clearance behind the elbow
- Fixed init failing check-states on arm3_Link/chassis_link against the old
  radius
- Changed test_lesson_ik_target_is_reachable_over_a_band_of_pitches to
  ..._over_bands_of_pitches; arm3's extra travel opens a second, lower band
- Added _contiguous_bands (helper) to that test
- Documented that the wider bottom deck is unmodelled on purpose
- Removed the claim that the vendor init collides with the chassis

Co-Authored-By: Claude Opus 5 <noreply@anthropic.com>

File: dofbot_description/urdf/chassis.xacro (robot description, xacro)
@@ -16,5 +16,6 @@
   DOFBOT_FLOOR below.
   Defaults are the values measured on the real robot and validated at runtime
-  through the chassis_collision node (which this replaces).
+  through the chassis_collision node (which this replaces). The cylinder radius
+  is the pancake decks', not the body's widest point; see the note on it.
 -->
 <robot xmlns:xacro="http://www.ros.org/wiki/xacro">
@@ -36,7 +37,20 @@
   <xacro:property name="ground_drop"
                   value="${0.026 if floor_profile == 'hard' else 0.022}" />
+  <!-- Cylinder radius. This is the PANCAKE DECKS' radius, which is what the arm
+       can actually touch: level 2 sits at elbow height and every deck above it
+       is the same width. Set from a direct clearance measurement rather than a
+       tape across the body: at the 'init' fold, arm3_Link's rearmost point
+       sits 0.1646 m from the cylinder axis with 5 mm of air behind it, so the
+       decks reach 0.1596.
+       THE BOTTOM DECK IS WIDER THAN THIS AND IS DELIBERATELY NOT MODELLED. It
+       has a curved front and carries the bumpers, so it reaches out past every
+       deck above it, but it sits 3 mm above the arm's mounting plate and the
+       arm is never commanded into that space. One cylinder is one radius at
+       every height, so covering it would mean widening this number and taking
+       the 5 mm back off the elbow, which is the wrong trade; it needs its own
+       solid if it is ever modelled at all. -->
   <xacro:macro name="dofbot_chassis" params="
       parent:=base_link
-      radius:=0.165
+      radius:=0.1596
       height:=0.335
       back_offset:=0.265

File: dofbot_description/urdf/dofbot.urdf (robot description, URDF)
Before this commit: robot dofbot_description, 14 links, 13 joints
Joints:
- joint arm3_Joint: limit lower=-1.57 upper=1.57 effort=10 velocity=1000 -> lower=-1.57 upper=1.8850 effort=10 velocity=1000
