Commit message: increased the range of the base rotator to real world limits on robot

File: dofbot_description/urdf/dofbot.urdf (robot description, URDF)
Before this commit: robot dofbot_description, 14 links, 13 joints
Joints:
- joint arm1_Joint: limit lower=-1.57 upper=1.57 effort=10 velocity=1000 -> lower=-1.9024 upper=1.8850 effort=10 velocity=1000

Commit message: Correct shoulder height, joint limits, and grasp geometry
- Changed _D_BASE to 0.0745 (Z0 = 0.1075) for this arm's 32 mm standoffs
- Changed arm1_Joint origin to 0.0745 in the URDF for the same 18 mm
- Added JOINT_LIMITS (tuple) and in_limits (helper) per joint, replacing the
  single symmetric JOINT_LIMIT that clipped base yaw to +-90 and ignored the
  wider arm1 range already present in the URDF
- Changed ik, moveit_client, and pick_place limit checks to use JOINT_LIMITS
- Added measured tip offsets to gripper._TABLE, computed from the Rlink2 mesh
- Removed the collision-search _hover in favour of tip_offset_for lookup
- Changed pick_place pitch sweep to pi/2..pi at 0.01 rad, nearest-first
- Added reach-versus-posture diagnosis to the no-approach error
- Added convex-hull collision meshes for arm1..arm4 and make_collision_meshes
  (tool) that builds them
- Changed base_link collision to a box and cylinder primitive pair
- Added a powered-off-arm check to moveit_bridge and port-contention
  detection to joint_state_mirror
- Changed mirror.rviz RobotModel durability to Transient Local and added a
  collision-geometry RobotModel
- Updated named-state TCP heights in NAMED_STATES and the SRDF for the new Z0
- Added tests for URDF limit transcription, the 217 deg yaw sector, in_limits,
  and tip-offset sign

File: dofbot_description/urdf/dofbot.urdf (robot description, URDF)
Before this commit: robot dofbot_description, 14 links, 13 joints
Links:
- link arm1_Link: geometry collision mesh filename=package://dofbot_description/meshes/collision/arm1_Link.STL; visual mesh filename=package://dofbot_description/meshes/arm1_Link.STL
- link arm2_Link: geometry collision mesh filename=package://dofbot_description/meshes/collision/arm2_Link.STL; visual mesh filename=package://dofbot_description/meshes/arm2_Link.STL
- link arm3_Link: geometry collision mesh filename=package://dofbot_description/meshes/collision/arm3_Link.STL; visual mesh filename=package://dofbot_description/meshes/arm3_Link.STL
- link arm4_Link: geometry collision mesh filename=package://dofbot_description/meshes/collision/arm4_Link.STL; visual mesh filename=package://dofbot_description/meshes/arm4_Link.STL
- link base_link: geometry collision box size=0.1450 0.1200 0.0030; collision cylinder length=0.0770 radius=0.0400
Joints:
- joint arm1_Joint: origin xyz=0 0 0.0925 rpy=0 0 0 -> xyz=0 0 0.0745 rpy=0 0 0

Commit message: Shorten base_link mesh to match the physical standoffs
- Removed 18 mm of lower standoff from base_link.STL in Fusion, so the visual
  now agrees with arm1_Joint at 0.0745 and the collision primitives
- Reduced base_link.STL to 31,052 triangles from 116,335 and closed its holes,
  leaving 3 degenerate interior slivers from 1565 non-manifold edges
- Changed the base collision box origin to -0.0125 in x, correcting a 1 mm
  offset that left the plate corners outside it
- Changed the base collision cylinder to span z 0.0030..0.0828, covering the
  four servo screw heads standing proud of the housing shoulder
- Updated the standoff notes in dofbot.urdf, dofbot_kinematics, and
  make_collision_meshes, which promised a permanent visual/collision mismatch

File: dofbot_description/urdf/dofbot.urdf (robot description, URDF)
Before this commit: robot dofbot_description, 14 links, 13 joints
Links:
- link base_link: geometry collision box size=0.1450 0.1200 0.0030; collision cylinder length=0.0798 radius=0.0400
