Commit message: Fold init tighter and raise arm3's limit to the measured contact
- Changed init to a lower, tighter fold re-posed by hand on the arm
- Raised arm3_Joint's upper limit to where the arm's parts touch, in the URDF and JOINT_LIMITS
- Updated the startup positions to the new init
- Changed the near-edge and grip-height approach tests for the narrower strip and extra margin
- Changed the lesson IK test to expect one unbroken band of pitches

Co-Authored-By: Claude Opus 5.5 <noreply@anthropic.com>

File: dofbot_description/urdf/dofbot.urdf (robot description, URDF)
Before this commit: robot dofbot_description, 14 links, 13 joints
Joints:
- joint arm3_Joint: limit lower=-1.57 upper=1.8850 effort=10 velocity=1000 -> lower=-1.57 upper=2.2166 effort=10 velocity=1000
